File: kicad/hm-mod-rpi-rtc.sch (KiCad schematic (older format))
At the start: 12 parts, among them P1 RPI CONN, U1 DS3231

Commit message: v1.0
Parts:
- BT1: footprint (none) -> hm-mod-uart:CR1220_holder
- C2: value 100u -> 100u/10V; footprint (none) -> Capacitors_Tantalum_SMD:CP_Tantalum_Case-B_EIA-3528-21_Hand
- U1: footprint Housings_SOIC:SOIC-16_7.5x10.3mm_Pitch1.27mm -> Housings_SOIC:SOIC-16W_7.5x10.3mm_Pitch1.27mm
Changed lines of the file:
@@
 EESchema Schematic File Version 2
-LIBS:hm-mod-rpi-rtc-rescue
 LIBS:power
 LIBS:device
@@
 P 4550 1850
 F 0 "C2" H 4575 1950 50  0000 L CNN
-F 1 "100u" H 4500 1650 50  0000 L CNN
-F 2 "" H 4588 1700 50  0001 C CNN
+F 1 "100u/10V" H 4450 2150 50  0000 L CNN
+F 2 "Capacitors_Tantalum_SMD:CP_Tantalum_Case-B_EIA-3528-21_Hand" H 4588 1700 50  0001 C CNN
 F 3 "" H 4550 1850 50  0000 C CNN
 	1    4550 1850
@@
 F 0 "U1" H 2400 4675 50  0000 R CNN
 F 1 "DS3231" H 2400 4600 50  0000 R CNN
-F 2 "Housings_SOIC:SOIC-16_7.5x10.3mm_Pitch1.27mm" H 2550 3800 50  0001 L CNN
+F 2 "Housings_SOIC:SOIC-16W_7.5x10.3mm_Pitch1.27mm" H 2550 3800 50  0001 L CNN
 F 3 "" H 2770 4450 50  0001 C CNN
 	1    2500 4200
@@
 F 0 "BT1" H 3250 4850 50  0000 L CNN
 F 1 "CR1220" H 3250 4750 50  0000 L CNN
-F 2 "" V 3150 4810 50  0001 C CNN
+F 2 "hm-mod-uart:CR1220_holder" V 3150 4810 50  0001 C CNN
 F 3 "" V 3150 4810 50  0000 C CNN
 	1    3150 4750
